Commit message: Adding changes to arduino communication

File: src/robo2/urdf/robot2.xacro (robot description, xacro)
@@ -4,6 +4,22 @@
      For more information, please see http://wiki.ros.org/sw_urdf_exporter -->
 <robot xmlns:xacro="http://www.ros.org/wiki/xacro" >
-  <link
-    name="base_link">
+   <!-- BASE LINK -->
+    <link name="base_link">
+    </link>
+    <!-- BASE_FOOTPRINT LINK -->
+    <joint name="base_footprint_joint" type="fixed">
+        <parent link="base_link"/>
+        <child link="base_footprint"/>
+        <origin xyz="0 0 0" rpy="0 0 0"/>
+    </joint>
+    <link name="base_footprint">
+    </link>
+  <joint name="chassis_joint" type="fixed">
+        <parent link="base_link"/>
+        <child link="chassis_link"/>
+        <origin xyz="0 0 0"/>
+    </joint>
+  <link
+    name="chassis_link">
     <inertial>
       <origin
@@ -91,5 +107,5 @@
       rpy="-1.5708 0 0" />
     <parent
-      link="base_link" />
+      link="chassis_link" />
     <child
       link="rueda_izq_arriba" />
@@ -144,5 +160,5 @@
       rpy="-1.5708 0 0" />
     <parent
-      link="base_link" />
+      link="chassis_link" />
     <child
       link="rueda_izq_abajo" />
@@ -197,5 +213,5 @@
       rpy="1.5708 0 0" />
     <parent
-      link="base_link" />
+      link="chassis_link" />
     <child
       link="rueda_der_abajo" />
@@ -250,5 +266,5 @@
       rpy="1.5708 0 0" />
     <parent
-      link="base_link" />
+      link="chassis_link" />
     <child
       link="rueda_der_arriba" />
@@ -303,5 +319,5 @@
       rpy="0 0 0" />
     <parent
-      link="base_link" />
+      link="chassis_link" />
     <child
       link="lidar" />
